File: getting_to_blinky/getting_to_blinky.sch (KiCad schematic (older format))
At the start: 7 parts, among them U1 7555

Commit message: update
Parts:
- BT1: Spice_Model (none) -> dc 5; Spice_Netlist_Enabled (none) -> Y; Spice_Primitive (none) -> V
- D1: Spice_Lib_File (none) -> /Users/thomascountz/Documents/Projects/Personal/KiCad-Spice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; Spice_Model (none) -> LED_GENERAL; Spice_Netlist_Enabled (none) -> Y; Spice_Primitive (none) -> D
- U1: Spice_Lib_File (none) -> /Users/thomascountz/Documents/Projects/Personal/KiCad-Spice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; Spice_Model (none) -> NE555; Spice_Netlist_Enabled (none) -> Y; Spice_Primitive (none) -> X
Connections:
- net VDD: no longer names the net of BT1.1 (+), R1.1, U1.4 (RST), U1.8 (VDD)
Changed lines of the file:
@@
 F 2 "Package_SO:SOIC-8_3.9x4.9mm_P1.27mm" H 6200 3200 50  0001 C CNN
 F 3 "" H 6200 3200 50  0001 C CNN
+F 4 "X" H 6050 3750 50  0001 C CNN "Spice_Primitive"
+F 5 "NE555" H 6050 3750 50  0001 C CNN "Spice_Model"
+F 6 "Y" H 6050 3750 50  0001 C CNN "Spice_Netlist_Enabled"
+F 7 "/Users/thomascountz/Documents/Projects/Personal/KiCad-Spice-Library/Models/uncategorized/Bordodynovs Electronics Lib/sub/NE555.sub" H 6050 3750 50  0001 C CNN "Spice_Lib_File"
 	1    6050 3750
 	1    0    0    -1
@@
 F 2 "LED_SMD:LED_0805_2012Metric_Pad1.15x1.40mm_HandSolder" H 6750 4450 50  0001 C CNN
 F 3 "~" H 6750 4450 50  0001 C CNN
+F 4 "D" H 6750 4450 50  0001 C CNN "Spice_Primitive"
+F 5 "LED_GENERAL" H 6750 4450 50  0001 C CNN "Spice_Model"
+F 6 "Y" H 6750 4450 50  0001 C CNN "Spice_Netlist_Enabled"
+F 7 "/Users/thomascountz/Documents/Projects/Personal/KiCad-Spice-Library/Models/Diode/led.lib" H 6750 4450 50  0001 C CNN "Spice_Lib_File"
 	1    6750 4450
 	0    -1   -1   0
@@
 F 2 "getting_to_blinky:S8211-46R" V 4550 4010 50  0001 C CNN
 F 3 "~" V 4550 4010 50  0001 C CNN
+F 4 "V" H 4550 3950 50  0001 C CNN "Spice_Primitive"
+F 5 "dc 5" H 4550 3950 50  0001 C CNN "Spice_Model"
+F 6 "Y" H 4550 3950 50  0001 C CNN "Spice_Netlist_Enabled"
 	1    4550 3950
 	1    0    0    -1
@@
 	5150 4700 5650 4700
 NoConn ~ 6150 4300
-Text Label 5350 3100 0    50   ~ 0
-VDD
 $EndSCHEMATC
