File: Hexo/Hexo.sch (KiCad schematic (older format))
At the start: 18 parts, among them Q1 BC557, SW1 SW_SPST, U1 LMC555xN, U2 4017

Commit message: add hexo files
Parts:
- removed SW1: SW_SPST, symbol Switch:SW_SPST
- removed U1: LMC555xN, Package_DIP:DIP-8_W7.62mm, symbol Timer:LMC555xN
- added SW1: SW_Push, Button_Switch_SMD:SW_SPST_TL3342, symbol Switch:SW_Push
- added SW2: SW_SPST, Button_Switch_SMD:SW_SPDT_CK-JS102011SAQN, symbol Switch:SW_SPST
- added U1: 7555, Package_SO:SOIC-8_3.9x4.9mm_P1.27mm, symbol Hexo:7555
- BT1: value Battery_Cell -> CR2032; footprint (none) -> Hexo:S8211-46R
- C1, C2: footprint (none) -> Capacitor_SMD:C_0805_2012Metric_Pad1.18x1.45mm_HandSolder
- D1, D2, D3, D4, D5, D6: footprint (none) -> LED_SMD:LED_0805_2012Metric_Pad1.15x1.40mm_HandSolder
- Q1: value BC557 -> BC857; footprint Package_TO_SOT_THT:TO-92_Inline -> Package_TO_SOT_SMD:SOT-23; symbol Transistor_BJT:BC557 -> Transistor_BJT:BC857
- R1, R2, R3, R4, R5: footprint (none) -> Resistor_SMD:R_0805_2012Metric_Pad1.20x1.40mm_HandSolder
- U2: value 4017 -> 74HC4017; footprint (none) -> Package_SO:SOIC-16_3.9x9.9mm_P1.27mm
Connections:
- net GND: now also SW1.2, SW2.2 (B), U1.1 (GND); no longer BT1.2 (-)
- net VCC: now also Q1.2 (E), U1.4 (~R), U1.8 (VCC); no longer Q1.3 (E)
- net at R1.1, R3.2: now also Q1.1 (B); no longer Q1.2 (B)
- net at C1.2, R1.2: now also SW1.1
- net at R4.1: now also Q1.3 (C); no longer Q1.1 (C)
- net at C2.1, R2.1, R4.2: now also U1.2 (TRG), U1.6 (THR), U1.7 (DIS)
- net at U2.14 (CLK): now also U1.3 (OUT)
- net at D6.1 (K): now also D1.1 (K), D2.1 (K), D3.1 (K), D4.1 (K), D5.1 (K), R5.1; no longer U2.1 (Q5)
- net at U2.10 (Q4): now also D5.2 (A); no longer D5.1 (K)
- net at U2.2 (Q1): now also D2.2 (A); no longer D2.1 (K)
- net at U2.3 (Q0): now also D1.2 (A); no longer D1.1 (K)
- net at U2.4 (Q2): now also D3.2 (A); no longer D3.1 (K)
- net at U2.7 (Q3): now also D4.2 (A); no longer D4.1 (K)
- new net: D6.2 (A), U2.1 (Q5)
- new net: BT1.2 (-), SW2.1 (A)
Other:
- moved on the sheet: BT1, C1, C2, D1, D2, D3, D4, D5, D6, Q1, R1, R2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
